Commit message: Add base_link definition

File: src/description/sam_bot_description.urdf (robot description, URDF)
Before this commit: robot sam_bot, 0 links, 0 joints
Links:
- added link base_link; visual box size=${base_length} ${base_width} ${base_height}

Commit message: Add base_joint

File: src/description/sam_bot_description.urdf (robot description, URDF)
Before this commit: robot sam_bot, 2 links, 0 joints
Joints:
- added joint base_joint: type fixed, parent base_link, child , origin xyz=0.0 0.0 ${-(wheel_radius+wheel_zoff)} rpy=0 0 0

Commit message: Add wheels description

File: src/description/sam_bot_description.urdf (robot description, URDF)
Before this commit: robot sam_bot, 2 links, 1 joints
Joints:
- joint base_joint: origin xyz=0.0 0.0 ${-(wheel_radius+wheel_zoff)} rpy=0 0 0 -> xyz=0.0 0.0 ${-(wheel_radius + wheel_zoff)} rpy=0 0 0

Commit message: Add castor wheel link

File: src/description/sam_bot_description.urdf (robot description, URDF)
Before this commit: robot sam_bot, 2 links, 1 joints
Links:
- added link front_caster; visual sphere radius=${(wheel_radius + wheel_zoff - (base_height / 2.0))}

Commit message: Add caster_joint description

File: src/description/sam_bot_description.urdf (robot description, URDF)
Before this commit: robot sam_bot, 3 links, 1 joints
Joints:
- added joint caster_joint: type fixed, parent base_link, child front_caster, origin xyz=${caster_xoff} 0.0 ${-(base_height / 2.0)} rpy=0 0 0
