Commit message: Error fixes

File: src/sam_bot_description/src/description/sam_bot_description.urdf (robot description, URDF)
Before this commit: robot sam_bot, 3 links, 2 joints
Joints:
- joint base_joint: child  -> base_footprint

Commit message: Add collision areas to front_caster

File: src/sam_bot_description/src/description/sam_bot_description.urdf (robot description, URDF)
Before this commit: robot sam_bot, 3 links, 2 joints
Links:
- link front_caster: geometry collision sphere radius=${(wheel_radius+wheel_zoff-(base_height/2))}; visual sphere radius=${(wheel_radius + wheel_zoff - (base_height / 2.0))}

Commit message: Add imu_link

File: src/sam_bot_description/src/description/sam_bot_description.urdf (robot description, URDF)
Before this commit: robot sam_bot, 3 links, 2 joints
Links:
- added link imu_link; visual box 

Commit message: Add collision areas to imu_link

File: src/sam_bot_description/src/description/sam_bot_description.urdf (robot description, URDF)
Before this commit: robot sam_bot, 4 links, 2 joints
Links:
- link imu_link: geometry collision box ; visual box 
